File: dancebots-pcb/dancebots-pcb.sch (KiCad schematic (older format))
At the start: 33 parts, among them J1 BATTERY, J2 MOT2-L, J3 MOT1-R, J4 MP3 Player, U1 L4941, U2 L293, U3 ATTINY861A-P, U4 LM386, U5 LM358

Commit message: version 7.0 sent off for prototyping
Parts:
- C2: footprint Capacitors_THT:CP_Radial_D7.5mm_P2.50mm -> dancebots_fp:ELcap4.1mm
- C4, C5, C6, C8, C9: footprint (none) -> dancebots_fp:CAPC
- C7: footprint (none) -> dancebots_fp:ElCap_6.4mm
- D0: footprint (none) -> LEDs:LED_D5.0mm
- J1: footprint (none) -> dancebots_fp:BATT
- J4: footprint (none) -> dancebots_fp:MP3
- LED0, LED1, LED2, LED3, LED4, LED5, LED6, LED7: footprint (none) -> dancebots_fp:LED
- R1, R2, R3: footprint (none) -> dancebots_fp:RES
- RN1, RN2: footprint Resistors_THT:R_Array_SIP8 -> dancebots_fp:RN
- U1: footprint Power_Integrations:TO-220 -> dancebots_fp:TO-220
- U2: footprint (none) -> Housings_DIP:DIP-16_W7.62mm_LongPads
- U3: footprint (none) -> Housings_DIP:DIP-20_W7.62mm_LongPads
- U4, U5: footprint (none) -> Housings_DIP:DIP-8_W7.62mm_LongPads
Connections:
- net GND: now also D0.1 (K)
- net at D0.2 (A): now also R1.2
Other:
- moved on the sheet: D0
Changed lines of the file:
@@
 Title "Dancebots PCB"
 Date "2017-08-17"
-Rev "v6.0"
+Rev "v7.0"
 Comp "RoboMINT"
-Comment1 "Credits to Raymond Oung for V1.0 - V5.0, this design is a transfer of V6.0 to KiCAD"
+Comment1 "Credits to Raymond Oung for V1.0 - V6.0, this design is a transfer of V6.0 to KiCAD"
 Comment2 ""
 Comment3 ""
@@
 F 0 "U4" H 8800 2250 50  0000 L CNN
 F 1 "LM386" H 8800 2150 50  0000 L CNN
-F 2 "" H 8850 2050 50  0001 C CNN
+F 2 "Housings_DIP:DIP-8_W7.62mm_LongPads" H 8850 2050 50  0001 C CNN
 F 3 "" H 8950 2150 50  0000 C CNN
 F 4 "000" H 8750 1950 60  0001 C CNN "PN"
@@
 F 0 "U2" H 1775 4775 60  0000 C CNN
 F 1 "L293" H 1825 4675 60  0000 C CNN
-F 2 "" H 2075 4225 60  0001 C CNN
+F 2 "Housings_DIP:DIP-16_W7.62mm_LongPads" H 2075 4225 60  0001 C CNN
 F 3 "" H 2075 4225 60  0000 C CNN
 	1    2075 4225
@@
 F 0 "U1" H 1525 2075 50  0000 C CNN
 F 1 "L4941" H 1725 2075 50  0000 L CNN
-F 2 "Power_Integrations:TO-220" H 1725 1975 50  0001 C CIN
+F 2 "dancebots_fp:TO-220" H 1725 1975 50  0001 C CIN
 F 3 "" H 1725 1875 50  0000 C CNN
 F 4 "000" H 1725 1875 60  0001 C CNN "PN"
@@
 L LED D0
 U 1 1 5995DBB6
-P 2900 2125
-F 0 "D0" H 2900 2225 50  0000 C CNN
-F 1 "PWR" H 2900 2025 50  0000 C CNN
-F 2 "" H 2900 2125 50  0001 C CNN
-F 3 "" H 2900 2125 50  0000 C CNN
-	1    2900 2125
+P 2900 2075
+F 0 "D0" H 2900 2175 50  0000 C CNN
+F 1 "PWR" H 2900 1975 50  0000 C CNN
+F 2 "LEDs:LED_D5.0mm" H 2900 2075 50  0001 C CNN
+F 3 "" H 2900 2075 50  0000 C CNN
+	1    2900 2075
 	0    -1   -1   0
 $EndComp
@@
 F 0 "R1" V 2980 1775 50  0000 C CNN
 F 1 "150" V 2900 1775 50  0000 C CNN
-F 2 "" V 2830 1775 50  0001 C CNN
+F 2 "dancebots_fp:RES" V 2830 1775 50  0001 C CNN
 F 3 "" H 2900 1775 50  0000 C CNN
 	1    2900 1775
@@
 F 0 "C2" H 2275 2075 50  0000 L CNN
 F 1 "22uF" H 2275 1875 50  0000 L CNN
-F 2 "Capacitors_THT:CP_Radial_D7.5mm_P2.50mm" H 2250 1975 50  0001 C CNN
+F 2 "dancebots_fp:ELcap4.1mm" H 2250 1975 50  0001 C CNN
 F 3 "" H 2250 1975 50  0000 C CNN
 	1    2250 1975
@@
 F 0 "U3" H 4800 3025 50  0000 C CNN
 F 1 "ATTINY861A-P" H 6450 1125 50  0000 C CNN
-F 2 "" H 5750 2075 50  0000 C CIN
+F 2 "Housings_DIP:DIP-20_W7.62mm_LongPads" H 5750 2075 50  0001 C CIN
 F 3 "" H 5700 2075 50  0000 C CNN
 	1    5700 2075
@@
 F 0 "C4" H 4375 1525 50  0000 L CNN
 F 1 "100nF" H 4375 1325 50  0000 L CNN
-F 2 "" H 4388 1275 50  0001 C CNN
+F 2 "dancebots_fp:CAPC" H 4388 1275 50  0001 C CNN
 F 3 "" H 4350 1425 50  0000 C CNN
 	1    4350 1425
@@
 F 0 "C5" V 8775 1350 50  0000 L CNN
 F 1 "100nF" V 8850 1350 50  0000 L CNN
-F 2 "" H 9038 1250 50  0001 C CNN
+F 2 "dancebots_fp:CAPC" H 9038 1250 50  0001 C CNN
 F 3 "" H 9000 1400 50  0000 C CNN
 F 4 "000" H 9000 1400 60  0001 C CNN "PN"
@@
 F 0 "C9" H 10000 2200 50  0000 L CNN
 F 1 "10pF" H 10000 2000 50  0000 L CNN
-F 2 "" H 10013 1950 50  0001 C CNN
+F 2 "dancebots_fp:CAPC" H 10013 1950 50  0001 C CNN
 F 3 "" H 9975 2100 50  0000 C CNN
 F 4 "000" H 9975 2100 60  0001 C CNN "PN"
@@
 F 0 "C7" H 9550 2050 50  0000 L CNN
 F 1 "220uF" H 9550 1850 50  0000 L CNN
-F 2 "" H 9525 1950 50  0001 C CNN
+F 2 "dancebots_fp:ElCap_6.4mm" H 9525 1950 50  0001 C CNN
 F 3 "" H 9525 1950 50  0000 C CNN
 F 4 "000" H 9525 1950 60  0001 C CNN "PN"
@@
 F 0 "U5" H 8875 4875 50  0000 L CNN
 F 1 "LM358" H 8875 4425 50  0000 L CNN
-F 2 "" H 8925 4675 50  0001 C CNN
+F 2 "Housings_DIP:DIP-8_W7.62mm_LongPads" H 8925 4675 50  0001 C CNN
 F 3 "" H 8925 4675 50  0000 C CNN
 F 4 "000" H 8925 4675 60  0001 C CNN "PN"
@@
 F 0 "C8" V 9200 4125 50  0000 L CNN
 F 1 "100nF" V 9125 4000 50  0000 L CNN
-F 2 "" H 9013 4075 50  0001 C CNN
+F 2 "dancebots_fp:CAPC" H 9013 4075 50  0001 C CNN
 F 3 "" H 8975 4225 50  0000 C CNN
 	1    8975 4225
@@
 F 0 "R3" V 9605 2250 50  0000 C CNN
 F 1 "10" V 9525 2250 50  0000 C CNN
-F 2 "" V 9455 2250 50  0001 C CNN
+F 2 "dancebots_fp:RES" V 9455 2250 50  0001 C CNN
 F 3 "" H 9525 2250 50  0000 C CNN
 F 4 "000" H 9525 2250 60  0001 C CNN "PN"
@@
 F 0 "R2" V 9355 2800 50  0000 C CNN
 F 1 "10k" V 9275 2800 50  0000 C CNN
-F 2 "" V 9205 2800 50  0001 C CNN
+F 2 "dancebots_fp:RES" V 9205 2800 50  0001 C CNN
 F 3 "" H 9275 2800 50  0000 C CNN
 F 4 "000" H 9275 2800 60  0001 C CNN "PN"
@@
 F 0 "C6" H 9075 2475 50  0000 L CNN
 F 1 "47nF" H 9000 2550 50  0000 L CNN
-F 2 "" H 9313 2350 50  0001 C CNN
+F 2 "dancebots_fp:CAPC" H 9313 2350 50  0001 C CNN
 F 3 "" H 9275 2500 50  0000 C CNN
 F 4 "000" H 9275 2500 60  0001 C CNN "PN"
@@
 F 0 "LED0" H 900 7250 50  0000 C CNN
 F 1 "LED" H 900 7050 50  0000 C CNN
-F 2 "" H 900 7150 50  0001 C CNN
+F 2 "dancebots_fp:LED" H 900 7150 50  0001 C CNN
 F 3 "" H 900 7150 50  0001 C CNN
 	1    900  7150
@@
 F 0 "LED1" H 1200 7250 50  0000 C CNN
 F 1 "LED" H 1200 7050 50  0000 C CNN
-F 2 "" H 1200 7150 50  0001 C CNN
+F 2 "dancebots_fp:LED" H 1200 7150 50  0001 C CNN
 F 3 "" H 1200 7150 50  0001 C CNN
 	1    1200 7150
@@
 F 0 "LED2" H 1500 7250 50  0000 C CNN
 F 1 "LED" H 1500 7050 50  0000 C CNN
-F 2 "" H 1500 7150 50  0001 C CNN
+F 2 "dancebots_fp:LED" H 1500 7150 50  0001 C CNN
 F 3 "" H 1500 7150 50  0001 C CNN
 	1    1500 7150
@@
 F 0 "LED3" H 1800 7250 50  0000 C CNN
 F 1 "LED" H 1800 7050 50  0000 C CNN
-F 2 "" H 1800 7150 50  0001 C CNN
+F 2 "dancebots_fp:LED" H 1800 7150 50  0001 C CNN
 F 3 "" H 1800 7150 50  0001 C CNN
 	1    1800 7150
@@
 F 0 "LED4" H 2200 7250 50  0000 C CNN
 F 1 "LED" H 2200 7050 50  0000 C CNN
-F 2 "" H 2200 7150 50  0001 C CNN
+F 2 "dancebots_fp:LED" H 2200 7150 50  0001 C CNN
 F 3 "" H 2200 7150 50  0001 C CNN
 	1    2200 7150
@@
 F 0 "LED5" H 2500 7250 50  0000 C CNN
 F 1 "LED" H 2500 7050 50  0000 C CNN
-F 2 "" H 2500 7150 50  0001 C CNN
+F 2 "dancebots_fp:LED" H 2500 7150 50  0001 C CNN
 F 3 "" H 2500 7150 50  0001 C CNN
 	1    2500 7150
@@
 F 0 "LED6" H 2800 7250 50  0000 C CNN
 F 1 "LED" H 2800 7050 50  0000 C CNN
-F 2 "" H 2800 7150 50  0001 C CNN
+F 2 "dancebots_fp:LED" H 2800 7150 50  0001 C CNN
 F 3 "" H 2800 7150 50  0001 C CNN
 	1    2800 7150
@@
 F 0 "LED7" H 3100 7250 50  0000 C CNN
 F 1 "LED" H 3100 7050 50  0000 C CNN
-F 2 "" H 3100 7150 50  0001 C CNN
+F 2 "dancebots_fp:LED" H 3100 7150 50  0001 C CNN
 F 3 "" H 3100 7150 50  0001 C CNN
 	1    3100 7150
@@
 F 0 "RN1" V 700 6550 50  0000 C CNN
 F 1 "82" V 1900 6550 50  0000 C CNN
-F 2 "Resistors_THT:R_Array_SIP8" V 1975 6550 50  0001 C CNN
+F 2 "dancebots_fp:RN" V 1975 6550 50  0001 C CNN
 F 3 "" H 1300 6550 50  0001 C CNN
 	1    1300 6550
@@
 F 0 "RN2" V 2000 6550 50  0000 C CNN
 F 1 "82" V 3200 6550 50  0000 C CNN
-F 2 "Resistors_THT:R_Array_SIP8" V 3275 6550 50  0001 C CNN
+F 2 "dancebots_fp:RN" V 3275 6550 50  0001 C CNN
 F 3 "" H 2600 6550 50  0001 C CNN
 	1    2600 6550
@@
 L GND #PWR024
 U 1 1 59BEB876
-P 2900 2325
-F 0 "#PWR024" H 2900 2075 50  0001 C CNN
-F 1 "GND" H 2900 2175 50  0000 C CNN
-F 2 "" H 2900 2325 50  0000 C CNN
-F 3 "" H 2900 2325 50  0000 C CNN
-	1    2900 2325
+P 2900 2225
+F 0 "#PWR024" H 2900 1975 50  0001 C CNN
+F 1 "GND" H 2900 2075 50  0000 C CNN
+F 2 "" H 2900 2225 50  0000 C CNN
+F 3 "" H 2900 2225 50  0000 C CNN
+	1    2900 2225
 	1    0    0    -1
 $EndComp
@@
 F 0 "J4" H 5100 4600 50  0000 C CNN
 F 1 "MP3 Player" V 5200 4400 50  0000 C CNN
-F 2 "" H 5100 4400 50  0001 C CNN
+F 2 "dancebots_fp:MP3" H 5100 4400 50  0001 C CNN
 F 3 "" H 5100 4400 50  0001 C CNN
 	1    5100 4400
@@
 F 0 "J1" H 5100 6600 50  0000 C CNN
 F 1 "BATTERY" V 5200 6450 50  0000 C CNN
-F 2 "" H 5100 6450 50  0001 C CNN
+F 2 "dancebots_fp:BATT" H 5100 6450 50  0001 C CNN
 F 3 "" H 5100 6450 50  0001 C CNN
 	1    5100 6450

Commit message: v7.2: fixed symbol and library references, added part numbers, and cleaned up gnd vias on PCB
Parts:
- C1, C3, C4, C8: symbol C -> Device:C; Lead Spacing (none) -> 5.08mm; Part Number (none) -> C322C104M5U5TA7301; Product Link (none) -> https://www.digikey.ch/products/en?keywords=399-9880-1-ND; Voltage Rating (none) -> 50V
- C2: symbol CP1 -> Device:CP1; Diameter (none) -> 4mm; Lead Spacing (none) -> 2mm; Part Number (none) -> 16MS522MEFC5X5; Product Link (none) -> https://www.digikey.com/product-detail/en/rubycon/16MS522ME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; Voltage Rating (none) -> 16V
- C5: symbol C -> Device:C; Lead Spacing (none) -> 5.08mm; PN 000 -> (none); Part Number (none) -> C322C104M5U5TA7301; Product Link (none) -> https://www.digikey.ch/products/en?keywords=399-9880-1-ND; Voltage Rating (none) -> 50V
- C6: symbol C -> Device:C; Lead Spacing (none) -> 5.08mm; PN 000 -> (none); Part Number (none) -> C322C473K5R5TA7301; Product Link (none) -> https://www.digikey.ch/products/en?keywords=399-13939-1-ND; Voltage Rating (none) -> 50V
- C7: symbol CP1 -> Device:CP1; Diameter (none) -> 6.3mm; Lead Spacing (none) -> 2.5mm; PN 000 -> (none); Part Number (none) -> 16YXJ220MT16.3X11; Product Link (none) -> https://www.digikey.ch/products/en?keywords=1189-1546-1-ND; Voltage Rating (none) -> 16V
- C9: symbol C -> Device:C; Lead Spacing (none) -> 5.08mm; PN 000 -> (none); Part Number (none) -> C317C100J5G5TA; Product Link (none) -> https://www.digikey.ch/products/en?keywords=399-8910-ND%09; Voltage Rating (none) -> 50V
- D0: footprint LEDs:LED_D5.0mm -> LED_THT:LED_D5.0mm; symbol LED -> Device:LED; Lead Spacing (none) -> 2.54mm; Product Link (none) -> https://www.sparkfun.com/products/9662
- J1: symbol CONN_01X02 -> Connector_Generic:Conn_01x02; Lead Spacing (none) -> 2.54mm; Part Number (none) -> SBH341AS; Product Link (none) -> https://www.digikey.com/products/en?keywords=SBH-341AS
- J2, J3: symbol CONN_01X02 -> Connector_Generic:Conn_01x02; Additional Component (none) -> https://www.sparkfun.com/products/9914; Lead Spacing (none) -> 2mm; Part Number (none) -> S2B-PH-K-S; Product Link (none) -> https://www.digikey.com/products/en?keywords=455-1719-ND
- J4: symbol CONN_01X03 -> Connector_Generic:Conn_01x03; Part Number (none) -> CA-2207; Product Link (none) -> https://www.digikey.com/products/en?keywords=CP-2207-ND%09
- JP18: symbol CONN_01X02 -> Connector_Generic:Conn_01x02; Additional Component (none) -> https://www.sparkfun.com/products/9914; Lead Spacing (none) -> 2mm; PN 000 -> (none); Part Number (none) -> S2B-PH-K-S; Product Link (none) -> https://www.digikey.com/products/en?keywords=455-1719-ND
- LED0, LED1, LED2, LED3, LED4, LED5, LED6, LED7: symbol LED -> Device:LED; Diameter (none) -> 5mm; Lead Spacing (none) -> 2.54mm; Product Link (none) -> https://www.sparkfun.com/products/9662
- R1: symbol R -> Device:R; Lead Spacing (none) -> 10.16mm; Part Number (none) -> CF14JT150R; Power Rating (none) -> 0.25W; Product Link (none) -> https://www.digikey.com/products/en?keywords=CF14JT150RCT-ND
- R2: symbol R -> Device:R; Lead Spacing (none) -> 10.16mm; PN 000 -> (none); Part Number (none) -> CF14JT10K0; Power Rating (none) -> 0.25W; Product Link (none) -> https://www.digikey.com/products/en?keywords=CF14JT10K0CT-ND
- R3: symbol R -> Device:R; Lead Spacing (none) -> 10.16mm; PN 000 -> (none); Part Number (none) -> CF14JT10R0; Power Rating (none) -> 0.25W; Product Link (none) -> https://www.digikey.com/products/en?keywords=CF14JT10R0CT-ND
- RN1, RN2: symbol R_Pack04_SIP -> Device:R_Pack04_SIP; Lead Spacing (none) -> 2.54mm; Part Number (none) -> 4608X-102-820LF; Power Rating (none) -> 0.3W; Product Link (none) -> https://www.digikey.com/products/en?keywords=4608X-2-820LF-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
- U1: symbol LM7809CT -> dancebots-parts:L4941; Lead Spacing (none) -> 2.54mm; PN 000 -> (none); Part Number (none) -> L4941BV; Product Link (none) -> https://www.digikey.com/products/en?keywords=497-6695-5-ND
- U2: footprint Housings_DIP:DIP-16_W7.62mm_LongPads -> Package_DIP:DIP-16_W7.62mm_LongPads; symbol L293 -> dancebots-parts:L293; Additional Component (none) -> https://www.digikey.com/products/en?keywords=A120349-ND; Lead Spacing (none) -> 2.54mm; Part Number (none) -> L293D; Product Link (none) -> https://www.digikey.com/products/en?keywords=497-2936-5-ND%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
- U3: value ATTINY861A-P -> ATTINY261A-P; footprint Housings_DIP:DIP-20_W7.62mm_LongPads -> Package_DIP:DIP-20_W7.62mm_LongPads; symbol ATTINY861A-P -> dancebots-parts:ATTINY261A-P; Additional Component (none) -> https://www.digikey.com/products/en?keywords=A120351-ND; Lead Spacing (none) -> 2.54mm; Part Number (none) -> ATTINY261A-PU; Product Link (none) -> https://www.digikey.com/products/en?keywords=ATTINY261A-PU-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
- U4: footprint Housings_DIP:DIP-8_W7.62mm_LongPads -> Package_DIP:DIP-8_W7.62mm_LongPads; symbol LM386 -> dancebots-parts:LM386; Additional Component (none) -> https://www.digikey.com/products/en?keywords=A120347-ND; Lead Spacing (none) -> 2.54mm; PN 000 -> (none); Part Number (none) -> LM386N-4/NOPB; Product Link (none) -> https://www.digikey.com/products/en?keywords=296-43960-5-ND
- U5: footprint Housings_DIP:DIP-8_W7.62mm_LongPads -> Package_DIP:DIP-8_W7.62mm_LongPads; symbol LM358 -> dancebots-parts:LM358; Additional Component (none) -> https://www.digikey.com/products/en?keywords=A120347-ND; Lead Spacing (none) -> 2.54mm; PN 000 -> (none); Part Number (none) -> LM358P; Product Link (none) -> https://www.digikey.com/products/en?keywords=296-1395-5-ND
