File: dancebots-pcb/dancebots-pcb.kicad_pcb (KiCad board)
At the start: 2 copper layers, 50 x 61 mm, 38 parts, among them J1 BATTERY, J2 MOT2-L, J3 MOT1-R, U1 L4941, U2 L293, U3 ATTINY261A-P, U4 LM386, U5 LM358, U6 DFR0299

Commit message: Minor change: Version on Silkscreen
Other:
- board text added: "MP3 DanceBot V8.2 mint & pepper 2022"
- board text removed: "MP3 DanceBot V8.1 mint & pepper 2022"
Changed lines of the file:
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@@
     (effects (font (size 1.1 1.1) (thickness 0.17)) (justify left mirror))
   )
-  (gr_text "MP3 DanceBot V8.1\nmint & pepper 2022" (at 137.1 114) (layer "B.SilkS")
+  (gr_text "MP3 DanceBot V8.2\nmint & pepper 2022" (at 137.1 114) (layer "B.SilkS")
     (effects (font (size 1.1 1.1) (thickness 0.17)) (justify left mirror))
   )

Commit message: updated mcu to attiny861 in schematic and pcb; migrated to kicad v7
Parts:
- U3: value ATTINY261A-P -> ATTINY861A-P
Other:
- board text added: "MP3 DanceBot V8.3 mint & pepper 2025"
- board text removed: "MP3 DanceBot V8.2 mint & pepper 2022"
